Commit message: major simulation changes and sensor implementations

File: sim_car/urdf/car.urdf (robot description, URDF)
Before this commit: robot sim_car, 8 links, 7 joints
Links:
- added link steering_fl_link, mass 0.5; visual box size=0.04 0.04 0.05
- added link steering_fr_link, mass 0.5; visual box size=0.04 0.04 0.05
- added link suspension_fl_link, mass 2.0; visual box size=0.05 0.05 0.15
- added link suspension_fr_link, mass 2.0; visual box size=0.05 0.05 0.15
- added link suspension_rl_link, mass 2.0; visual box size=0.05 0.05 0.15
- added link suspension_rr_link, mass 2.0; visual box size=0.05 0.05 0.15
- link base_link: mass 10.0 -> 200.0; geometry collision box size=2.0 0.8 0.15; visual box size=2.0 0.8 0.15
- link front_left_wheel: mass 0.5 -> 8.0; geometry collision cylinder length=0.18 radius=0.23; visual cylinder length=0.18 radius=0.23
- link front_right_wheel: mass 0.5 -> 8.0; geometry collision cylinder length=0.18 radius=0.23; visual cylinder length=0.18 radius=0.23
- link gps_link: mass 0.01 -> 0.02; geometry visual cylinder length=0.02 radius=0.03
- link imu_link: mass 0.01 -> 0.05; geometry visual box size=0.04 0.04 0.02
- link rear_left_wheel: mass 0.5 -> 10.0; geometry collision cylinder length=0.20 radius=0.23; visual cylinder length=0.20 radius=0.23
- link rear_right_wheel: mass 0.5 -> 10.0; geometry collision cylinder length=0.20 radius=0.23; visual cylinder length=0.20 radius=0.23
Joints:
- added joint steering_fl_joint: type revolute, parent suspension_fl_link, child steering_fl_link, origin xyz=0 0 -0.05 rpy=0 0 0, axis 0 0 1, limit lower=-0.52 upper=0.52 effort=100 velocity=3.0
- added joint steering_fr_joint: type revolute, parent suspension_fr_link, child steering_fr_link, origin xyz=0 0 -0.05 rpy=0 0 0, axis 0 0 1, limit lower=-0.52 upper=0.52 effort=100 velocity=3.0
- added joint suspension_fl_joint: type prismatic, parent base_link, child suspension_fl_link, origin xyz=0.8 0.55 -0.1 rpy=0 0 0, axis 0 0 1, limit lower=-0.05 upper=0.05 effort=10000 velocity=1.0
- added joint suspension_fr_joint: type prismatic, parent base_link, child suspension_fr_link, origin xyz=0.8 -0.55 -0.1 rpy=0 0 0, axis 0 0 1, limit lower=-0.05 upper=0.05 effort=10000 velocity=1.0
- added joint suspension_rl_joint: type prismatic, parent base_link, child suspension_rl_link, origin xyz=-0.8 0.55 -0.1 rpy=0 0 0, axis 0 0 1, limit lower=-0.05 upper=0.05 effort=10000 velocity=1.0
- added joint suspension_rr_joint: type prismatic, parent base_link, child suspension_rr_link, origin xyz=-0.8 -0.55 -0.1 rpy=0 0 0, axis 0 0 1, limit lower=-0.05 upper=0.05 effort=10000 velocity=1.0
- joint base_joint: origin xyz=0.0 0.0 0.1 rpy=0 0 0 -> xyz=0.0 0.0 0.25 rpy=0 0 0
- joint front_left_wheel_joint: origin xyz=0.2 0.225 -0.1 rpy=0 0 0 -> xyz=0 0.05 -0.08 rpy=0 0 0; parent base_link -> steering_fl_link
- joint front_right_wheel_joint: origin xyz=0.2 -0.225 -0.1 rpy=0 0 0 -> xyz=0 -0.05 -0.08 rpy=0 0 0; parent base_link -> steering_fr_link
- joint gps_joint: origin xyz=-0.2 0 0.15 rpy=0 0 0 -> xyz=-0.5 0 0.15 rpy=0 0 0
- joint imu_joint: origin xyz=0 0 0 rpy=0 0 0 -> xyz=0 0 0.1 rpy=0 0 0
- joint rear_left_wheel_joint: origin xyz=-0.2 0.225 -0.1 rpy=0 0 0 -> xyz=0 0.05 -0.13 rpy=0 0 0; parent base_link -> suspension_rl_link
- joint rear_right_wheel_joint: origin xyz=-0.2 -0.225 -0.1 rpy=0 0 0 -> xyz=0 -0.05 -0.13 rpy=0 0 0; parent base_link -> suspension_rr_link

Commit message: merged plotting with eufs

File: sim_car/urdf/car.urdf (robot description, URDF)
Before this commit: robot sim_car, 14 links, 13 joints
Links:
- link base_link: geometry collision mesh filename=package://sim_car/meshes/sisu-20d.dae; visual mesh filename=package://sim_car/meshes/sisu-20d.dae
- link front_left_wheel: geometry collision mesh filename=package://sim_car/meshes/wheel_left.dae; visual mesh filename=package://sim_car/meshes/wheel_left.dae
- link front_right_wheel: geometry collision mesh filename=package://sim_car/meshes/wheel_right.dae; visual mesh filename=package://sim_car/meshes/wheel_right.dae
- link rear_left_wheel: geometry collision mesh filename=package://sim_car/meshes/wheel_left.dae; visual mesh filename=package://sim_car/meshes/wheel_left.dae
- link rear_right_wheel: geometry collision mesh filename=package://sim_car/meshes/wheel_right.dae; visual mesh filename=package://sim_car/meshes/wheel_right.dae
