Commit message: added cameras

File: sim_car/urdf/eufs_car.urdf.xacro (robot description, xacro)
@@ -4,4 +4,7 @@
   <xacro:arg name="chassis_mesh" default="file://$(find sim_car)/meshes/sisu-20d.dae"/>
   <xacro:arg name="topic_prefix" default="/sim/raw"/>
+  <xacro:arg name="publish_track_cones" default="true"/>
+  <xacro:arg name="enable_cone_miscoloring" default="false"/>
+  <xacro:arg name="cone_confusion_yaml" default="$(find gazebo_cone_plugins)/config/cone_confusion_matrix.yaml"/>
   <xacro:property name="config" value="${load_yaml('$(arg config_file)')}"/>
   <material name="tire_mat">
@@ -54,4 +57,39 @@
     <origin xyz="-0.5 0 0.15" rpy="0 0 0"/>
   </joint>
+  <!-- Stereo Camera Links -->
+  <link name="stereo_left_link">
+    <visual>
+      <geometry>
+        <box size="0.04 0.03 0.02"/>
+      </geometry>
+      <material name="silver"/>
+    </visual>
+    <inertial>
+      <mass value="0.03"/>
+      <inertia ixx="0.00001" ixy="0.0" ixz="0.0" iyy="0.00001" iyz="0.0" izz="0.00001"/>
+    </inertial>
+  </link>
+  <joint name="stereo_left_joint" type="fixed">
+    <parent link="chassis"/>
+    <child link="stereo_left_link"/>
+    <origin xyz="1.71 0.06 0.2" rpy="0 0 0"/>
+  </joint>
+  <link name="stereo_right_link">
+    <visual>
+      <geometry>
+        <box size="0.04 0.03 0.02"/>
+      </geometry>
+      <material name="silver"/>
+    </visual>
+    <inertial>
+      <mass value="0.03"/>
+      <inertia ixx="0.00001" ixy="0.0" ixz="0.0" iyy="0.00001" iyz="0.0" izz="0.00001"/>
+    </inertial>
+  </link>
+  <joint name="stereo_right_joint" type="fixed">
+    <parent link="chassis"/>
+    <child link="stereo_right_link"/>
+    <origin xyz="1.71 -0.06 0.2" rpy="0 0 0"/>
+  </joint>
   <!-- EUFS dynamics plugin (gz-sim) -->
   <gazebo>
@@ -73,4 +111,29 @@
     </plugin>
   </gazebo>
+  <!-- Remastered cone plugin (Ignition Gazebo Fortress) -->
+  <gazebo>
+    <plugin filename="libgazebo_ground_truth_cones.so"
+            name="gazebo_plugins::eufs_plugins::GazeboGroundTruthConesRemastered">
+      <updateRate>100.0</updateRate>
+      <trackModelName>track</trackModelName>
+      <carFrameLink>base_footprint</carFrameLink>
+      <groundTruthTrackTopicName>/ground_truth/track</groundTruthTrackTopicName>
+      <visibleConesTopicName>/ground_truth/cones</visibleConesTopicName>
+      <trackFrame>map</trackFrame>
+      <visibleFrame>base_footprint</visibleFrame>
+      <publishTrack>$(arg publish_track_cones)</publishTrack>
+      <cameraViewDistance>15.0</cameraViewDistance>
+      <cameraMinViewDistance>0.5</cameraMinViewDistance>
+      <cameraFOV>2.09</cameraFOV>
+      <lidarOn>true</lidarOn>
+      <lidarViewDistance>100.0</lidarViewDistance>
+      <lidarMinViewDistance>1.0</lidarMinViewDistance>
+      <lidarXViewDistance>20.0</lidarXViewDistance>
+      <lidarYViewDistance>20.0</lidarYViewDistance>
+      <lidarFOV>3.141593</lidarFOV>
+      <enableConeMiscoloring>$(arg enable_cone_miscoloring)</enableConeMiscoloring>
+      <confusionMatrixYaml>$(arg cone_confusion_yaml)</confusionMatrixYaml>
+    </plugin>
+  </gazebo>
   <!-- Joint State Publisher -->
   <gazebo>
@@ -173,3 +236,49 @@
     </sensor>
   </gazebo>
+  <!-- Stereo Left Camera Sensor -->
+  <gazebo reference="stereo_left_link">
+    <sensor name="stereo_left_camera" type="camera">
+      <topic>$(arg topic_prefix)/stereo/left/image_raw</topic>
+      <camera_info_topic>$(arg topic_prefix)/stereo/left/camera_info</camera_info_topic>
+      <update_rate>15</update_rate>
+      <always_on>true</always_on>
+      <visualize>false</visualize>
+      <camera>
+        <!-- ZED 2i (2.1mm lens) -->
+        <horizontal_fov>1.919862</horizontal_fov>
+        <image>
+          <width>1920</width>
+          <height>1080</height>
+          <format>R8G8B8</format>
+        </image>
+        <clip>
+          <near>0.3</near>
+          <far>20.0</far>
+        </clip>
+      </camera>
+    </sensor>
+  </gazebo>
+  <!-- Stereo Right Camera Sensor -->
+  <gazebo reference="stereo_right_link">
+    <sensor name="stereo_right_camera" type="camera">
+      <topic>$(arg topic_prefix)/stereo/right/image_raw</topic>
+      <camera_info_topic>$(arg topic_prefix)/stereo/right/camera_info</camera_info_topic>
+      <update_rate>15</update_rate>
+      <always_on>true</always_on>
+      <visualize>false</visualize>
+      <camera>
+        <!-- ZED 2i (2.1mm lens) -->
+        <horizontal_fov>1.919862</horizontal_fov>
+        <image>
+          <width>1920</width>
+          <height>1080</height>
+          <format>R8G8B8</format>
+        </image>
+        <clip>
+          <near>0.3</near>
+          <far>20.0</far>
+        </clip>
+      </camera>
+    </sensor>
+  </gazebo>
 </robot>

Commit message: lidar implemented and works rmse

File: sim_car/urdf/eufs_car.urdf.xacro (robot description, xacro)
@@ -92,4 +92,22 @@
     <origin xyz="1.71 -0.06 0.2" rpy="0 0 0"/>
   </joint>
+  <!-- 2D LiDAR Sensor Link -->
+  <link name="lidar_link">
+    <visual>
+      <geometry>
+        <cylinder radius="0.04" length="0.05"/>
+      </geometry>
+      <material name="silver"/>
+    </visual>
+    <inertial>
+      <mass value="0.12"/>
+      <inertia ixx="0.00005" ixy="0.0" ixz="0.0" iyy="0.00005" iyz="0.0" izz="0.00005"/>
+    </inertial>
+  </link>
+  <joint name="lidar_joint" type="fixed">
+    <parent link="chassis"/>
+    <child link="lidar_link"/>
+    <origin xyz="1.45 0 -0.09" rpy="0 0 0"/>
+  </joint>
   <!-- EUFS dynamics plugin (gz-sim) -->
   <gazebo>
@@ -282,3 +300,37 @@
     </sensor>
   </gazebo>
+  <!-- Front 270-degree 2D LiDAR Sensor -->
+  <gazebo reference="lidar_link">
+    <sensor name="front_lidar" type="gpu_lidar">
+      <topic>$(arg topic_prefix)/lidar</topic>
+      <update_rate>15</update_rate>
+      <always_on>true</always_on>
+      <visualize>false</visualize>
+      <lidar>
+        <scan>
+          <horizontal>
+            <samples>1080</samples>
+            <resolution>1</resolution>
+            <min_angle>-2.35619449</min_angle>
+            <max_angle>2.35619449</max_angle>
+          </horizontal>
+          <vertical>
+            <samples>1</samples>
+            <resolution>1</resolution>
+            <min_angle>0.0</min_angle>
+            <max_angle>0.0</max_angle>
+          </vertical>
+        </scan>
+        <range>
+          <min>0.10</min>
+          <max>30.0</max>
+          <resolution>0.01</resolution>
+        </range>
+        <noise type="gaussian">
+          <mean>0.0</mean>
+          <stddev>0.02</stddev>
+        </noise>
+      </lidar>
+    </sensor>
+  </gazebo>
 </robot>

Commit message: fixed wheelbaseframe for controlelr

File: sim_car/urdf/eufs_car.urdf.xacro (robot description, xacro)
@@ -312,6 +312,6 @@
             <samples>1080</samples>
             <resolution>1</resolution>
-            <min_angle>-2.26892803</min_angle>
-            <max_angle>2.26892803</max_angle>
+            <min_angle>-1.91986218</min_angle>
+            <max_angle>1.91986218</max_angle>
           </horizontal>
           <vertical>

File: sim_car/urdf/eufs_wheels.urdf.xacro (robot description, xacro)
@@ -10,4 +10,10 @@
     <xacro:property name="wheel_friction_kp" value="1e8"/>
     <xacro:property name="steering_hinge_mass" value="1"/>
+    <link name="front_axle"/>
+    <joint name="front_axle_joint" type="fixed">
+      <parent link="chassis"/>
+      <child link="front_axle"/>
+      <origin xyz="${wheelbase / 2} 0 0" rpy="0 0 0"/>
+    </joint>
     <xacro:macro name="wheel" params="lr_prefix fr_prefix">
       <link name="${lr_prefix}_${fr_prefix}_wheel">

Commit message: added 3d lidar

File: sim_car/urdf/eufs_car.urdf.xacro (robot description, xacro)
@@ -7,8 +7,10 @@
   <xacro:arg name="perception_rate_hz" default="60.0"/>
   <xacro:arg name="planner_rate_hz" default="60.0"/>
+  <xacro:arg name="lidar_pipeline" default="pointcloud3d"/>
   <xacro:arg name="publish_track_cones" default="true"/>
   <xacro:arg name="enable_cone_miscoloring" default="false"/>
   <xacro:arg name="cone_confusion_yaml" default="$(find gazebo_cone_plugins)/config/cone_confusion_matrix.yaml"/>
-  <xacro:property name="config" value="${load_yaml('$(arg config_file)')}"/>
+  <xacro:property name="config" value="${xacro.load_yaml('$(arg config_file)')}"/>
+  <xacro:property name="lidar_pipeline_mode" value="$(arg lidar_pipeline)"/>
   <material name="tire_mat">
     <color rgba="0.05 0.05 0.05 1"/>
@@ -95,6 +97,6 @@
     <origin xyz="1.71 -0.06 0.2" rpy="0 0 0"/>
   </joint>
-  <!-- 2D LiDAR Sensor Link -->
-  <link name="lidar_link">
+  <!-- Legacy 2D LiDAR Sensor Link -->
+  <link name="lidar_scan_link">
     <visual>
       <geometry>
@@ -108,8 +110,26 @@
     </inertial>
   </link>
-  <joint name="lidar_joint" type="fixed">
-    <parent link="chassis"/>
-    <child link="lidar_link"/>
+  <joint name="lidar_scan_joint" type="fixed">
+    <parent link="chassis"/>
+    <child link="lidar_scan_link"/>
     <origin xyz="1.45 0 -0.09" rpy="0 0 0"/>
+  </joint>
+  <!-- OS1-style 3D LiDAR Sensor Link -->
+  <link name="lidar_os1_link">
+    <visual>
+      <geometry>
+        <cylinder radius="0.04" length="0.05"/>
+      </geometry>
+      <material name="silver"/>
+    </visual>
+    <inertial>
+      <mass value="0.12"/>
+      <inertia ixx="0.00005" ixy="0.0" ixz="0.0" iyy="0.00005" iyz="0.0" izz="0.00005"/>
+    </inertial>
+  </link>
+  <joint name="lidar_os1_joint" type="fixed">
+    <parent link="chassis"/>
+    <child link="lidar_os1_link"/>
+    <origin xyz="1.855 0 0.32" rpy="0 0 0"/>
   </joint>
   <!-- EUFS dynamics plugin (gz-sim) -->
@@ -303,37 +323,75 @@
     </sensor>
   </gazebo>
-  <!-- Front 260-degree 2D LiDAR Sensor -->
-  <gazebo reference="lidar_link">
-    <sensor name="front_lidar" type="gpu_lidar">
-      <topic>$(arg topic_prefix)/lidar</topic>
-      <update_rate>$(arg perception_rate_hz)</update_rate>
-      <always_on>true</always_on>
-      <visualize>false</visualize>
-      <lidar>
-        <scan>
-          <horizontal>
-            <samples>1080</samples>
-            <resolution>1</resolution>
-            <min_angle>-1.91986218</min_angle>
-            <max_angle>1.91986218</max_angle>
-          </horizontal>
-          <vertical>
-            <samples>1</samples>
-            <resolution>1</resolution>
-            <min_angle>0.0</min_angle>
-            <max_angle>0.0</max_angle>
-          </vertical>
-        </scan>
-        <range>
-          <min>0.10</min>
-          <max>30.0</max>
-          <resolution>0.01</resolution>
-        </range>
-        <noise type="gaussian">
-          <mean>0.0</mean>
-          <stddev>0.02</stddev>
-        </noise>
-      </lidar>
-    </sensor>
-  </gazebo>
+  <xacro:if value="${lidar_pipeline_mode == 'scan2d'}">
+    <!-- Legacy front 260-degree 2D LiDAR Sensor -->
+    <gazebo reference="lidar_scan_link">
+      <sensor name="front_lidar" type="gpu_lidar">
+        <topic>$(arg topic_prefix)/lidar</topic>
+        <update_rate>$(arg perception_rate_hz)</update_rate>
+        <always_on>true</always_on>
+        <visualize>false</visualize>
+        <lidar>
+          <scan>
+            <horizontal>
+              <samples>1080</samples>
+              <resolution>1</resolution>
+              <min_angle>-1.91986218</min_angle>
+              <max_angle>1.91986218</max_angle>
+            </horizontal>
+            <vertical>
+              <samples>1</samples>
+              <resolution>1</resolution>
+              <min_angle>0.0</min_angle>
+              <max_angle>0.0</max_angle>
+            </vertical>
+          </scan>
+          <range>
+            <min>0.10</min>
+            <max>30.0</max>
+            <resolution>0.01</resolution>
+          </range>
+          <noise type="gaussian">
+            <mean>0.0</mean>
+            <stddev>0.02</stddev>
+          </noise>
+        </lidar>
+      </sensor>
+    </gazebo>
+  </xacro:if>
+  <xacro:unless value="${lidar_pipeline_mode == 'scan2d'}">
+    <!-- OS1-like 3D LiDAR profile -->
+    <gazebo reference="lidar_os1_link">
+      <sensor name="front_lidar" type="gpu_lidar">
+        <topic>$(arg topic_prefix)/lidar</topic>
+        <update_rate>10.0</update_rate>
+        <always_on>true</always_on>
+        <visualize>false</visualize>
+        <lidar>
+          <scan>
+            <horizontal>
+              <samples>1024</samples>
+              <resolution>1</resolution>
+              <min_angle>-3.14159265</min_angle>
+              <max_angle>3.14159265</max_angle>
+            </horizontal>
+            <vertical>
+              <samples>32</samples>
+              <resolution>1</resolution>
+              <min_angle>-0.3700098</min_angle>
+              <max_angle>0.3700098</max_angle>
+            </vertical>
+          </scan>
+          <range>
+            <min>0.50</min>
+            <max>50.0</max>
+            <resolution>0.01</resolution>
+          </range>
+          <noise type="gaussian">
+            <mean>0.0</mean>
+            <stddev>0.02</stddev>
+          </noise>
+        </lidar>
+      </sensor>
+    </gazebo>
+  </xacro:unless>
 </robot>

Commit message: refractor lidar3d

File: sim_car/urdf/eufs_car.urdf.xacro (robot description, xacro)
@@ -13,4 +13,21 @@
   <xacro:property name="config" value="${xacro.load_yaml('$(arg config_file)')}"/>
   <xacro:property name="lidar_pipeline_mode" value="$(arg lidar_pipeline)"/>
+  <xacro:property name="lidar_scan_mount_xyz" value="1.45 0 -0.09"/>
+  <xacro:property name="lidar_os1_mount_xyz" value="1.855 0 0.32"/>
+  <xacro:property name="legacy_lidar_update_rate_hz" value="$(arg perception_rate_hz)"/>
+  <xacro:property name="legacy_lidar_horizontal_samples" value="1080"/>
+  <xacro:property name="legacy_lidar_min_angle_rad" value="-1.91986218"/>
+  <xacro:property name="legacy_lidar_max_angle_rad" value="1.91986218"/>
+  <xacro:property name="legacy_lidar_range_min_m" value="0.10"/>
+  <xacro:property name="legacy_lidar_range_max_m" value="30.0"/>
+  <xacro:property name="os1_lidar_update_rate_hz" value="10.0"/>
+  <xacro:property name="os1_lidar_horizontal_samples" value="2048"/>
+  <xacro:property name="os1_lidar_vertical_samples" value="32"/>
+  <xacro:property name="os1_lidar_min_angle_rad" value="-3.14159265"/>
+  <xacro:property name="os1_lidar_max_angle_rad" value="3.14159265"/>
+  <xacro:property name="os1_lidar_vertical_min_angle_rad" value="-0.3700098"/>
+  <xacro:property name="os1_lidar_vertical_max_angle_rad" value="0.3700098"/>
+  <xacro:property name="os1_lidar_range_min_m" value="0.50"/>
+  <xacro:property name="os1_lidar_range_max_m" value="50.0"/>
   <material name="tire_mat">
     <color rgba="0.05 0.05 0.05 1"/>
@@ -113,5 +130,5 @@
     <parent link="chassis"/>
     <child link="lidar_scan_link"/>
-    <origin xyz="1.45 0 -0.09" rpy="0 0 0"/>
+    <origin xyz="${lidar_scan_mount_xyz}" rpy="0 0 0"/>
   </joint>
   <!-- OS1-style 3D LiDAR Sensor Link -->
@@ -131,5 +148,5 @@
     <parent link="chassis"/>
     <child link="lidar_os1_link"/>
-    <origin xyz="1.855 0 0.32" rpy="0 0 0"/>
+    <origin xyz="${lidar_os1_mount_xyz}" rpy="0 0 0"/>
   </joint>
   <!-- EUFS dynamics plugin (gz-sim) -->
@@ -324,9 +341,9 @@
   </gazebo>
   <xacro:if value="${lidar_pipeline_mode == 'scan2d'}">
-    <!-- Legacy front 260-degree 2D LiDAR Sensor -->
+    <!-- Legacy 2D LiDAR profile kept intact for scan2d mode. -->
     <gazebo reference="lidar_scan_link">
       <sensor name="front_lidar" type="gpu_lidar">
         <topic>$(arg topic_prefix)/lidar</topic>
-        <update_rate>$(arg perception_rate_hz)</update_rate>
+        <update_rate>${legacy_lidar_update_rate_hz}</update_rate>
         <always_on>true</always_on>
         <visualize>false</visualize>
@@ -334,8 +351,8 @@
           <scan>
             <horizontal>
-              <samples>1080</samples>
+              <samples>${legacy_lidar_horizontal_samples}</samples>
               <resolution>1</resolution>
-              <min_angle>-1.91986218</min_angle>
-              <max_angle>1.91986218</max_angle>
+              <min_angle>${legacy_lidar_min_angle_rad}</min_angle>
+              <max_angle>${legacy_lidar_max_angle_rad}</max_angle>
             </horizontal>
             <vertical>
@@ -347,6 +364,6 @@
           </scan>
           <range>
-            <min>0.10</min>
-            <max>30.0</max>
+            <min>${legacy_lidar_range_min_m}</min>
+            <max>${legacy_lidar_range_max_m}</max>
             <resolution>0.01</resolution>
           </range>
@@ -360,9 +377,9 @@
   </xacro:if>
   <xacro:unless value="${lidar_pipeline_mode == 'scan2d'}">
-    <!-- OS1-like 3D LiDAR profile -->
+    <!-- OS1-like 3D LiDAR profile used only in pointcloud3d mode. -->
     <gazebo reference="lidar_os1_link">
       <sensor name="front_lidar" type="gpu_lidar">
         <topic>$(arg topic_prefix)/lidar</topic>
-        <update_rate>10.0</update_rate>
+        <update_rate>${os1_lidar_update_rate_hz}</update_rate>
         <always_on>true</always_on>
         <visualize>false</visualize>
@@ -370,19 +387,19 @@
           <scan>
             <horizontal>
-              <samples>2048</samples>
+              <samples>${os1_lidar_horizontal_samples}</samples>
               <resolution>1</resolution>
-              <min_angle>-3.14159265</min_angle>
-              <max_angle>3.14159265</max_angle>
+              <min_angle>${os1_lidar_min_angle_rad}</min_angle>
+              <max_angle>${os1_lidar_max_angle_rad}</max_angle>
             </horizontal>
             <vertical>
-              <samples>32</samples>
+              <samples>${os1_lidar_vertical_samples}</samples>
               <resolution>1</resolution>
-              <min_angle>-0.3700098</min_angle>
-              <max_angle>0.3700098</max_angle>
+              <min_angle>${os1_lidar_vertical_min_angle_rad}</min_angle>
+              <max_angle>${os1_lidar_vertical_max_angle_rad}</max_angle>
             </vertical>
           </scan>
           <range>
-            <min>0.50</min>
-            <max>50.0</max>
+            <min>${os1_lidar_range_min_m}</min>
+            <max>${os1_lidar_range_max_m}</max>
             <resolution>0.01</resolution>
           </range>
